File: hardware/hardware-py-a1/numcalcium.kicad_sch (KiCad schematic)
At the start: 2 parts, among them J1 Conn_01x14_Socket, J2 Conn_01x14_Socket

Commit message: hw: fixes for py-a1
Other:
- moved on the sheet: J1, J2
Changed lines of the file:
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@@
 	(symbol
 		(lib_id "Connector:Conn_01x14_Socket")
-		(at 213.36 76.2 0)
+		(at 198.12 69.85 90)
 		(unit 1)
 		(exclude_from_sim no)
@@
 		(dnp no)
 		(property "Reference" "J1"
-			(at 211.582 58.166 0)
+			(at 180.086 71.628 0)
 			(effects
 				(font
@@
 		)
 		(property "Value" "Conn_01x14_Socket"
-			(at 222.25 89.916 90)
+			(at 211.836 60.96 90)
 			(effects
 				(font
@@
 		)
 		(property "Footprint" "Connector_FFC-FPC:Hirose_FH12-14S-0.5SH_1x14-1MP_P0.50mm_Horizontal"
-			(at 213.36 76.2 0)
+			(at 198.12 69.85 0)
 			(effects
 				(font
@@
 		)
 		(property "Datasheet" "~"
-			(at 213.36 76.2 0)
+			(at 198.12 69.85 0)
 			(effects
 				(font
@@
 		)
 		(property "Description" "Generic connector, single row, 01x14, script generated"
-			(at 213.36 76.2 0)
+			(at 198.12 69.85 0)
 			(effects
 				(font
@@
 	(symbol
 		(lib_id "Connector:Conn_01x14_Socket")
-		(at 220.98 76.2 0)
-		(mirror y)
+		(at 198.12 67.31 90)
+		(mirror x)
 		(unit 1)
 		(exclude_from_sim no)
@@
 		(dnp no)
 		(property "Reference" "J2"
-			(at 223.012 57.912 0)
+			(at 179.832 65.278 0)
 			(effects
 				(font
@@
 		)
 		(property "Value" "Conn_01x14_Socket"
-			(at 219.71 78.7399 0)
+			(at 200.6599 68.58 0)
 			(effects
 				(font
@@
 		)
 		(property "Footprint" "Connector_FFC-FPC:Hirose_FH12-14S-0.5SH_1x14-1MP_P0.50mm_Horizontal"
-			(at 220.98 76.2 0)
+			(at 198.12 67.31 0)
 			(effects
 				(font
@@
 		)
 		(property "Datasheet" "~"
-			(at 220.98 76.2 0)
+			(at 198.12 67.31 0)
 			(effects
 				(font
@@
 		)
 		(property "Description" "Generic connector, single row, 01x14, script generated"
-			(at 220.98 76.2 0)
+			(at 198.12 67.31 0)
 			(effects
 				(font
@@
 	)
 	(sheet
-		(at 226.06 58.42)
-		(size 22.86 38.1)
-		(fields_autoplaced yes)
+		(at 168.91 41.91)
+		(size 62.23 20.32)
 		(stroke
 			(width 0.1524)
@@
 		)
 		(property "Sheetname" "Front"
-			(at 226.06 57.7084 0)
+			(at 168.656 64.516 0)
 			(effects
 				(font
@@
 		)
 		(property "Sheetfile" "front.kicad_sch"
-			(at 226.06 97.1046 0)
+			(at 231.7246 62.23 90)
 			(effects
 				(font
@@
 		)
 		(pin "LCD_DC" input
-			(at 226.06 78.74 180)
+			(at 200.66 62.23 270)
 			(effects
 				(font
@@
 		)
 		(pin "CK" input
-			(at 226.06 73.66 180)
+			(at 195.58 62.23 270)
 			(effects
 				(font
@@
 		)
 		(pin "MOSI" input
-			(at 226.06 71.12 180)
+			(at 193.04 62.23 270)
 			(effects
 				(font
@@
 		)
 		(pin "SD_CS" input
-			(at 226.06 76.2 180)
+			(at 198.12 62.23 270)
 			(effects
 				(font
@@
 		)
 		(pin "LCD_CS" input
-			(at 226.06 66.04 180)
+			(at 187.96 62.23 270)
 			(effects
 				(font
@@
 		)
 		(pin "LCD_LED" input
-			(at 226.06 81.28 180)
+			(at 203.2 62.23 270)
 			(effects
 				(font
@@
 		)
 		(pin "VDD" input
-			(at 226.06 60.96 180)
+			(at 182.88 62.23 270)
 			(effects
 				(font
@@
 		)
 		(pin "MISO" input
-			(at 226.06 68.58 180)
+			(at 190.5 62.23 270)
 			(effects
 				(font
@@
 		)
 		(pin "GND" input
-			(at 226.06 93.98 180)
+			(at 215.9 62.23 270)
 			(effects
 				(font
@@
 		)
 		(pin "A_R1" input
-			(at 226.06 91.44 180)
+			(at 213.36 62.23 270)
 			(effects
 				(font
@@
 		)
 		(pin "A_T" input
-			(at 226.06 88.9 180)
+			(at 210.82 62.23 270)
 			(effects
 				(font
@@
 		)
 		(pin "BUZZER" input
-			(at 226.06 83.82 180)
+			(at 205.74 62.23 270)
 			(effects
 				(font
@@
 		)
 		(pin "LED" input
-			(at 226.06 86.36 180)
+			(at 208.28 62.23 270)
 			(effects
 				(font
@@
 		)
 		(pin "LED_RETURN" input
-			(at 226.06 63.5 180)
+			(at 185.42 62.23 270)
 			(effects
 				(font
@@
 	)
 	(sheet
-		(at 146.05 58.42)
+		(at 168.91 74.93)
 		(size 62.23 96.52)
-		(fields_autoplaced yes)
 		(stroke
 			(width 0.1524)
@@
 		)
 		(property "Sheetname" "Main"
-			(at 146.05 57.7084 0)
+			(at 168.91 74.2184 0)
 			(effects
 				(font
@@
 		)
 		(property "Sheetfile" "main.kicad_sch"
-			(at 146.05 155.5246 0)
+			(at 232.156 94.742 90)
 			(effects
 				(font
@@
 		)
 		(pin "MOSI" input
-			(at 208.28 71.12 0)
+			(at 193.04 74.93 90)
 			(effects
 				(font
@@
 		)
 		(pin "LCD_CS" input
-			(at 208.28 66.04 0)
+			(at 187.96 74.93 90)
 			(effects
 				(font
@@
 		)
 		(pin "CK" input
-			(at 208.28 73.66 0)
+			(at 195.58 74.93 90)
 			(effects
 				(font
@@
 		)
 		(pin "MISO" input
-			(at 208.28 68.58 0)
+			(at 190.5 74.93 90)
 			(effects
 				(font
@@
 		)
 		(pin "SD_CS" input
-			(at 208.28 76.2 0)
+			(at 198.12 74.93 90)
 			(effects
 				(font
@@
 		)
 		(pin "LCD_DC" input
-			(at 208.28 78.74 0)
+			(at 200.66 74.93 90)
 			(effects
 				(font
@@
 		)
 		(pin "LCD_LED" input
-			(at 208.28 81.28 0)
+			(at 203.2 74.93 90)
 			(effects
 				(font
@@
 		)
 		(pin "STATUS_LED" input
-			(at 208.28 86.36 0)
+			(at 208.28 74.93 90)
 			(effects
 				(font
@@
 		)
 		(pin "GND" input
-			(at 208.28 93.98 0)
+			(at 215.9 74.93 90)
 			(effects
 				(font
@@
 		)
 		(pin "VDD" input
-			(at 208.28 60.96 0)
+			(at 182.88 74.93 90)
 			(effects
 				(font
@@
 		)
 		(pin "BUZ_DRIVE" input
-			(at 208.28 83.82 0)
+			(at 205.74 74.93 90)
 			(effects
 				(font
@@
 		)
 		(pin "AUD_L" input
-			(at 208.28 88.9 0)
+			(at 210.82 74.93 90)
 			(effects
 				(font
@@
 		)
 		(pin "AUD_R" input
-			(at 208.28 91.44 0)
+			(at 213.36 74.93 90)
 			(effects
 				(font
@@
 		)
 		(pin "LED_RETURN" input
-			(at 208.28 63.5 0)
-			(effects
-				(font
+			(at 185.42 74.93 90)
+			(effects
+				(font
